Commit message: 10-robot ground position exchange: fake_sim and sensorless-Gazebo modes
Two run_sim.py modes drive ten Pioneer 3-ATs swapping positions on a
circle with the full planner->MPC->unicycle chain per robot:
multiagent-ground-fake (RViz only) and multiagent-ground-gazebo (real
P3AT models; use_lidar:=false use_camera:=false strips the 36k-ray
mid360 per robot — gzserver ~10% of one core for ten robots).
map_source:=sensor_cloud feeds each planner from a sub-floor cloud grid
(z = -3 m) that keeps the map machinery alive in an obstacle-free world.

goal_monitor gains circle slots, antipodal + random_slot goal patterns
with stable per-namespace seeding, start staggering, stagnation redraws
(a goal drawn onto an occupied slot is rejected by the planner; without
the redraw the rejected robot parks and blocks its own slot — measured
800 s pin), and default-off slot claims (measured both ways: removing
same-slot contention waits raised simultaneous-mover density and
worsened fleet close passes 4-10x).

fake_sim renders ground markers, and its Gazebo teleport is now a single
in-flight async request — the old detached blocking thread per 10 ms
tick piled up until EAGAIN aborted the node at fleet scale.
--mpc-rate/--mpc-horizon expose the MPC pairing (laptop-safe 20/10
defaults; 40/20 measured right on a 48-core host).

File: urdf/p3at.urdf.xacro (robot description, xacro)
@@ -18,15 +18,27 @@
   <xacro:arg name="namespace" default="NX01" />
   <xacro:arg name="d435_range_max_depth" default="5.0" />
+  <!-- Sensor toggles. Defaults keep every existing mode's expansion
+       byte-identical. use_lidar:=false drops the mid360 ray sensor (36,000
+       rays @ 10 Hz per robot — the dominant per-robot Gazebo cost) and
+       use_camera:=false drops the four D435 camera sensors; the
+       multiagent-ground-gazebo swap runs 10 robots with both off and feeds
+       the planner from the sub-floor cloud instead (map_source param). -->
+  <xacro:arg name="use_lidar" default="true" />
+  <xacro:arg name="use_camera" default="true" />
   <xacro:include filename="$(find mighty)/urdf/pioneer3at_body.urdf.xacro" />
   <!-- Disabled: fake_sim handles teleport and TF for ground robot -->
   <!-- <xacro:p3at_gazebo_ext name="$(arg namespace)_red_rover" namespace="$(arg namespace)" /> -->
   <xacro:include filename="$(find ros2_livox_simulation)/urdf/mid360.xacro" />
-  <xacro:mid360 name="$(arg namespace)_livox" namespace="$(arg namespace)" parent="base_link" topic="mid360" lidar_update_rate="10" >
-    <origin xyz="0 0 1.0" rpy="0 0.3 0"/>
-  </xacro:mid360>
+  <xacro:if value="$(arg use_lidar)">
+    <xacro:mid360 name="$(arg namespace)_livox" namespace="$(arg namespace)" parent="base_link" topic="mid360" lidar_update_rate="10" >
+      <origin xyz="0 0 1.0" rpy="0 0.3 0"/>
+    </xacro:mid360>
+  </xacro:if>
   <xacro:include filename="$(find mighty)/urdf/_d435.urdf.xacro" />
-  <xacro:sensor_d435 name="$(arg namespace)_d435" topics_ns="$(arg namespace)" range_max_depth="$(arg d435_range_max_depth)" parent="base_link"
-                     publish_pointcloud="false" color_sensor_rate="5" depth_sensor_rate="15" depth_plugin_rate="15.0" color_plugin_rate="5.0">
-    <origin xyz="0.2 0.0 0.45" rpy="0 0 0"/>
-  </xacro:sensor_d435>
+  <xacro:if value="$(arg use_camera)">
+    <xacro:sensor_d435 name="$(arg namespace)_d435" topics_ns="$(arg namespace)" range_max_depth="$(arg d435_range_max_depth)" parent="base_link"
+                       publish_pointcloud="false" color_sensor_rate="5" depth_sensor_rate="15" depth_plugin_rate="15.0" color_plugin_rate="5.0">
+      <origin xyz="0.2 0.0 0.45" rpy="0 0 0"/>
+    </xacro:sensor_d435>
+  </xacro:if>
 </robot>
